File: pcb/UltraCIC-III.kicad_pcb (KiCad board)
At the start: 2 copper layers, 10.5 x 20.7 mm, 4 parts, among them J1 Conn_01x08, J2 Conn_01x08, U1 ATtiny25-20S, U2 ATtiny25-20P

Commit message: Updated PCB
Parts:
- U1: footprint Package_SO:SOIC-8W_5.3x5.3mm_P1.27mm -> Eigene:SOP-8-Wide
Routing:
- net PB1: track 5.73 -> 4.98 mm
- net GND: track 32.5 -> 33.2 mm
- net PB2: track 6.52 -> 7.26 mm
- net PB5: track 26.4 -> 25.7 mm
Other:
- board size 10.5 x 20.7 mm -> 10.7 x 20.7 mm
- board text added: "Fuses: H: 0xDF L: 0xC0"
- board text added: "cut for install"
- board text added: "v20221208"
- board text removed: "v20220516"
